File: l3/l3.kicad_pcb (KiCad board)
At the start: 2 copper layers, 137.5 x 129.1 mm, 23 parts, among them J1 Conn_01x04, SW1 SW_SPDT, SW2 SW_SPDT, SW3 SW_SPDT, SW4 SW_SPDT, U4 DEV-15583

Commit message: readd trace
Routing:
- net /SCLToF: track 260.6 -> 272.7 mm
Changed lines of the file:
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@@
+	)
+	(segment
+		(start 82.25 72.82)
+		(end 78.469744 76.600256)
+		(width 0.25)
+		(layer "B.Cu")
+		(net 6)
 	)
 	(segment
@@
 		(width 0.25)
 		(layer "B.Cu")
+		(net 6)
+	)
+	(segment
+		(start 82.25 66.069548)
+		(end 82.25 72.82)
+		(width 0.25)
+		(layer "B.Cu")
