File: l3/l3.kicad_pcb (KiCad board)
At the start: 2 copper layers, 137.5 x 129.1 mm, 23 parts, among them J1 Conn_01x04, J2 Conn_01x06, J3 Conn_01x06, J4 Conn_01x06, J5 Conn_01x06, SW1 SW_SPDT, SW2 SW_SPDT, SW3 SW_SPDT, SW4 SW_SPDT, U4 DEV-15583

Commit message: v2.0
l2 l3 done for print
Parts:
- renumbered SW3 to Cam, SW2 to ESP, SW4 to IMU, SW1 to Teensy
Routing:
- net SDAToF: track 233.5 -> 247.3 mm
- net SCLToF: track 259.3 -> 257.2 mm
Other:
- outline, holes or cut-outs redrawn
Changed lines of the file:
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@@
 			(at 0 -4.2 0)
 			(layer "F.SilkS")
+			(hide yes)
 			(effects
 				(font
@@
 			(at 0 -1.43 45)
 			(layer "F.SilkS")
+			(hide yes)
 			(effects
 				(font
@@
 		(layer "F.Cu")
 		(at 59.07 123.76 90)
-		(property "Reference" "SW2"
-			(at 0 -2.54 90)
+		(property "Reference" "ESP"
+			(at -0.63 -5.69 90)
 			(unlocked yes)
 			(layer "F.SilkS")
@@
 			(at 0 -4.2 0)
 			(layer "F.SilkS")
+			(hide yes)
 			(effects
 				(font
@@
 			(at 0 -2.33 90)
 			(layer "F.SilkS")
+			(hide yes)
 			(effects
 				(font
@@
 			(at -5.715 -19.685 90)
 			(layer "F.SilkS")
+			(hide yes)
 			(effects
 				(font
@@
 		(layer "F.Cu")
 		(at 66.85 123.76 90)
-		(property "Reference" "SW4"
-			(at 0 -2.54 90)
+		(property "Reference" "IMU"
+			(at 0.03 6.28 90)
 			(unlocked yes)
 			(layer "F.SilkS")
@@
 		(layer "F.Cu")
 		(at 59.07 134.54 90)
-		(property "Reference" "SW3"
-			(at 0 -2.54 90)
+		(property "Reference" "Cam"
+			(at 0.26 -5.91 90)
 			(unlocked yes)
 			(layer "F.SilkS")
@@
 			(at 0 -4.2 0)
 			(layer "F.SilkS")
+			(hide yes)
 			(effects
 				(font
@@
 			(at 0 -4.2 0)
 			(layer "F.SilkS")
+			(hide yes)
 			(effects
 				(font
@@
 			(at 0 -4.2 0)
 			(layer "F.SilkS")
+			(hide yes)
 			(effects
 				(font
@@
 		(layer "F.Cu")
 		(at 66.85 134.54 90)
-		(property "Reference" "SW1"
-			(at 0 -2.54 90)
+		(property "Reference" "Teensy"
+			(at 4.95 6.06 90)
 			(unlocked yes)
 			(layer "F.SilkS")
@@
 			(at 0 -2.33 0)
 			(layer "F.SilkS")
+			(hide yes)
 			(effects
 				(font
@@
 			(at 0 -2.33 0)
 			(layer "F.SilkS")
+			(hide yes)
 			(effects
 				(font
@@
 			(at 0 -4.2 0)
 			(layer "F.SilkS")
+			(hide yes)
 			(effects
 				(font
@@
 			(at 0 -4.2 0)
 			(layer "F.SilkS")
+			(hide yes)
 			(effects
 				(font
@@
 			(at 0 -4.2 0)
 			(layer "F.SilkS")
+			(hide yes)
 			(effects
 				(font
@@
 			(at 0 -1.43 45)
 			(layer "F.SilkS")
+			(hide yes)
 			(effects
 				(font
@@
 			(at 0 -2.33 90)
 			(layer "F.SilkS")
+			(hide yes)
 			(effects
 				(font
@@
 			(unlocked yes)
 			(layer "F.SilkS")
+			(hide yes)
 			(effects
 				(font
@@
 	)
 	(gr_arc
-		(start 69.579392 37.679352)
-		(mid 72.058146 36.613958)
-		(end 74.7315 36.249999)
+		(start 140.420608 37.676805)
+		(mid 105 165.349999)
+		(end 69.579392 37.676805)
 		(stroke
 			(width 0.2)
@@
 	)
 	(gr_line
-		(start 135.2685 36.249999)
-		(end 74.7315 36.249999)
+		(start 135.2685 36.247451)
+		(end 74.7315 36.247451)
 		(stroke
 			(width 0.2)
@@
 	)
 	(gr_arc
-		(start 140.420608 37.679352)
-		(mid 105 165.352548)
-		(end 69.579392 37.679352)
+		(start 135.2685 36.247451)
+		(mid 137.941853 36.611413)
+		(end 140.420608 37.676805)
+		(stroke
+			(width 0.2)
+			(type default)
+		)
+		(layer "Edge.Cuts")
+	)
+	(gr_line
+		(start 131.05466 66.121858)
+		(end 145.762713 53.780336)
+		(stroke
+			(width 0.2)
+			(type default)
+		)
+		(layer "Edge.Cuts")
+	)
+	(gr_line
+		(start 154.247509 63.892122)
+		(end 139.539456 76.233644)
 		(stroke
 			(width 0.2)
@@
 	)
 	(gr_arc
-		(start 135.2685 36.249999)
-		(mid 137.941853 36.613961)
-		(end 140.420608 37.679352)
+		(start 69.579392 37.676805)
+		(mid 72.058146 36.611411)
+		(end 74.7315 36.247451)
+		(stroke
+			(width 0.2)
+			(type default)
+		)
+		(layer "Edge.Cuts")
+	)
+	(gr_line
+		(start 139.539456 76.233644)
+		(end 131.05466 66.121858)
+		(stroke
+			(width 0.2)
+			(type default)
+		)
+		(layer "Edge.Cuts")
+	)
+	(gr_line
+		(start 145.762713 53.780336)
+		(end 154.247509 63.892122)
 		(stroke
 			(width 0.2)
@@
 	)
 	(segment
-		(start 150.33 101.102548)
-		(end 150.33 81.85)
-		(width 0.5)
-		(layer "B.Cu")
-		(net 3)
-	)
-	(segment
 		(start 65.54 90.202548)
 		(end 65.54 90.25)
@@
 	)
 	(segment
+		(start 145.19 80.34)
+		(end 139.61 80.34)
+		(width 0.5)
+		(layer "B.Cu")
+		(net 3)
+	)
+	(segment
+		(start 121.19 57.67)
+		(end 111.4 57.67)
+		(width 0.5)
+		(layer "B.Cu")
+		(net 3)
+	)
+	(segment
 		(start 56.5 128.83)
 		(end 59.07 126.26)
@@
 	)
 	(segment
+		(start 152.23 103.002548)
+		(end 150.33 101.102548)
+		(width 0.5)
+		(layer "B.Cu")
+		(net 3)
+	)
+	(segment
+		(start 127.74 68.47)
+		(end 127.74 64.22)
+		(width 0.5)
+		(layer "B.Cu")
+		(net 3)
+	)
+	(segment
 		(start 136.23 133.555)
 		(end 132.095 137.69)
@@
 	)
 	(segment
-		(start 126.15 57.67)
-		(end 111.4 57.67)
+		(start 150.33 85.48)
+		(end 145.19 80.34)
 		(width 0.5)
 		(layer "B.Cu")
@@
 	)
 	(segment
+		(start 150.33 101.102548)
+		(end 150.33 85.48)
+		(width 0.5)
+		(layer "B.Cu")
+		(net 3)
+	)
+	(segment
 		(start 136.23 133.555)
 		(end 152.23 117.555)
@@
 	)
 	(segment
-		(start 152.23 117.555)
-		(end 152.23 103.002548)
+		(start 139.61 80.34)
+		(end 127.74 68.47)
 		(width 0.5)
 		(layer "B.Cu")
@@
 	)
 	(segment
-		(start 56.5 134.47)
-		(end 56.5 128.83)
+		(start 152.23 117.555)
+		(end 152.23 103.002548)
 		(width 0.5)
 		(layer "B.Cu")
@@
 	)
 	(segment
-		(start 152.23 103.002548)
-		(end 150.33 101.102548)
+		(start 56.5 134.47)
+		(end 56.5 128.83)
 		(width 0.5)
 		(layer "B.Cu")
@@
 	)
 	(segment
-		(start 150.33 81.85)
-		(end 126.15 57.67)
+		(start 127.74 64.22)
+		(end 121.19 57.67)
 		(width 0.5)
 		(layer "B.Cu")
@@
 	)
 	(segment
-		(start 105.79 59.68)
-		(end 132.57 59.68)
+		(start 125.06 62.21)
+		(end 122.53 59.68)
+		(width 0.25)
+		(layer "F.Cu")
+		(net 5)
+	)
+	(segment
+		(start 139.76 80.01)
+		(end 125.06 65.31)
+		(width 0.25)
+		(layer "F.Cu")
+		(net 5)
+	)
+	(segment
+		(start 154.49 88.28)
+		(end 146.22 80.01)
+		(width 0.25)
+		(layer "F.Cu")
+		(net 5)
+	)
+	(segment
+		(start 154.49 93.122548)
+		(end 154.49 88.28)
 		(width 0.25)
 		(layer "F.Cu")
@@
 	)
 	(segment
-		(start 154.49 81.6)
+		(start 152.23 95.382548)
 		(end 154.49 93.122548)
 		(width 0.25)
@@
 	)
 	(segment
-		(start 103.78 57.67)
-		(end 105.79 59.68)
-		(width 0.25)
-		(layer "F.Cu")
-		(net 5)
-	)
-	(segment
 		(start 67.56 111.24972)
 		(end 64.10972 114.7)
@@
 	)
 	(segment
-		(start 132.57 59.68)
-		(end 154.49 81.6)
-		(width 0.25)
-		(layer "F.Cu")
-		(net 5)
-	)
-	(segment
 		(start 58.54 90.822548)
 		(end 65.54 97.822548)
@@
 	)
 	(segment
+		(start 125.06 65.31)
+		(end 125.06 62.21)
+		(width 0.25)
+		(layer "F.Cu")
+		(net 5)
+	)
+	(segment
+		(start 146.22 80.01)
+		(end 139.76 80.01)
+		(width 0.25)
+		(layer "F.Cu")
+		(net 5)
+	)
+	(segment
+		(start 105.79 59.68)
+		(end 103.78 57.67)
+		(width 0.25)
+		(layer "F.Cu")
+		(net 5)
+	)
+	(segment
 		(start 62.145235 76.316765)
 		(end 59.403235 76.316765)
@@
 	)
 	(segment
-		(start 154.49 93.122548)
-		(end 152.23 95.382548)
+		(start 122.53 59.68)
+		(end 105.79 59.68)
 		(width 0.25)
 		(layer "F.Cu")
@@
 	)
 	(segment
-		(start 108.54 55.45)
-		(end 106.32 57.67)
+		(start 152.23 97.922548)
+		(end 155.45 94.702548)
 		(width 0.25)
 		(layer "F.Cu")
@@
 	)
 	(segment
-		(start 155.81 94.342548)
-		(end 155.81 78.77)
+		(start 148.48 52.1)
+		(end 111.89 52.1)
 		(width 0.25)
 		(layer "F.Cu")
@@
 	)
 	(segment
-		(start 152.23 97.922548)
-		(end 155.81 94.342548)
+		(start 111.89 52.1)
+		(end 106.32 57.67)
 		(width 0.25)
 		(layer "F.Cu")
@@
 	)
 	(segment
-		(start 155.81 78.77)
-		(end 132.49 55.45)
+		(start 155.45 94.702548)
+		(end 155.45 59.07)
 		(width 0.25)
 		(layer "F.Cu")
@@
 	)
 	(segment
-		(start 132.49 55.45)
-		(end 108.54 55.45)
+		(start 155.45 59.07)
+		(end 148.48 52.1)
 		(width 0.25)
 		(layer "F.Cu")
@@
 	)
 	(group ""
-		(members "830066ea-2711-4d9b-8d64-ba6b1fbd4307" "94f8931c-5185-46ff-83e4-55c0b2587a4b"
-			"d0791157-cdb2-48ea-88a5-c0ee592a1cc5" "e608b6a6-f073-4641-873d-23f43ec24f1c"
+		(members "14e06b1b-3022-489e-bd05-f37cdd747799" "192454eb-3a18-4831-bf96-963eb8a468ab"
+			"1ffbbb85-6dee-495b-ad39-969edbe1f206" "5ca9052c-f03d-4a7b-b2a5-4b594d2ed7b0"
+			"7e24e4c4-63aa-4d1f-b9e6-e80889e8c897" "c2e4eaf6-2712-4fd5-a1b5-02303d6bdb14"
+			"db5602a7-a281-4f0e-9185-eec713af5111" "de72a3f8-0cb4-4356-a97b-ae37bbf4c670"
 		)
 	)
