File: 2024/l2/_autosave-l2.kicad_sch (KiCad schematic)
At the start: 6 parts, among them J1 Conn_01x04, J2 Conn_01x02, J3 Conn_01x04, U1 DEV-15583, U2 VNH5019A-E, U3 TLP175A

Commit message: 20/7 final
Parts:
- added R1: 1k, symbol Device:R
Connections:
- net PWM: now reaches U1.2
- net PWM: now also R1.1
- net at U2.7 (PWM): now also R1.2
Other:
- moved on the sheet: U3
Changed lines of the file:
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@@
+	(wire
+		(pts
+			(xy 193.04 52.07) (xy 203.2 52.07)
+		)
+		(stroke
+			(width 0)
+			(type default)
+		)
+	)
 	(wire
 		(pts
@@
 	(wire
 		(pts
-			(xy 74.93 78.74) (xy 77.47 78.74)
+			(xy 41.91 58.42) (xy 52.07 58.42)
 		)
 		(stroke
@@
 	(wire
 		(pts
-			(xy 118.11 21.59) (xy 128.27 21.59)
+			(xy 74.93 78.74) (xy 77.47 78.74)
 		)
 		(stroke
@@
 	(wire
 		(pts
-			(xy 72.39 78.74) (xy 74.93 78.74)
+			(xy 118.11 21.59) (xy 128.27 21.59)
 		)
 		(stroke
@@
 	(wire
 		(pts
-			(xy 193.04 46.99) (xy 203.2 46.99)
+			(xy 72.39 78.74) (xy 74.93 78.74)
 		)
 		(stroke
@@
 	(wire
 		(pts
-			(xy 118.11 24.13) (xy 128.27 24.13)
+			(xy 193.04 46.99) (xy 203.2 46.99)
 		)
 		(stroke
@@
 		)
 	)
+	(wire
+		(pts
+			(xy 118.11 24.13) (xy 128.27 24.13)
+		)
+		(stroke
+			(width 0)
+			(type default)
+		)
+	)
+	(label "PWM"
+		(at 193.04 52.07 0)
+		(fields_autoplaced yes)
+		(effects
+			(font
+				(size 1.27 1.27)
+			)
+			(justify left bottom)
+		)
+	)
 	(label "RXL3"
 		(at 182.88 24.13 0)
@@
 	(label "TXL3"
 		(at 193.04 67.31 0)
+		(fields_autoplaced yes)
+		(effects
+			(font
+				(size 1.27 1.27)
+			)
+			(justify left bottom)
+		)
+	)
+	(label "PWM"
+		(at 41.91 58.42 0)
 		(fields_autoplaced yes)
 		(effects
@@
 	)
 	(symbol
+		(lib_id "Device:R")
+		(at 55.88 58.42 90)
+		(unit 1)
+		(exclude_from_sim no)
+		(in_bom yes)
+		(on_board yes)
+		(dnp no)
+		(fields_autoplaced yes)
+		(property "Reference" "R1"
+			(at 55.88 52.07 90)
+			(effects
+				(font
+					(size 1.27 1.27)
+				)
+			)
+		)
+		(property "Value" "1k"
+			(at 55.88 54.61 90)
+			(effects
+				(font
+					(size 1.27 1.27)
+				)
+			)
+		)
+		(property "Footprint" ""
+			(at 55.88 60.198 90)
+			(effects
+				(font
+					(size 1.27 1.27)
+				)
+				(hide yes)
+			)
+		)
+		(property "Datasheet" "~"
+			(at 55.88 58.42 0)
+			(effects
+				(font
+					(size 1.27 1.27)
+				)
+				(hide yes)
+			)
+		)
+		(property "Description" "Resistor"
+			(at 55.88 58.42 0)
+			(effects
+				(font
+					(size 1.27 1.27)
+				)
+				(hide yes)
+			)
+		)
+		(pin "1"
+		)
+		(pin "2"
+		)
+		(instances
+			(project ""
+				(path "/6e23b0dc-b56a-4591-91ab-7fa94dae0df0"
+					(reference "R1")
+					(unit 1)
+				)
+			)
+		)
+	)
+	(symbol
 		(lib_id "power:GND")
 		(at 160.02 21.59 270)
@@
 	(symbol
 		(lib_id "Relay_SolidState:TLP175A")
-		(at 105.41 45.72 0)
+		(at 74.93 36.83 270)
 		(unit 1)
 		(exclude_from_sim no)
@@
 		(fields_autoplaced yes)
 		(property "Reference" "U3"
-			(at 105.41 36.83 0)
-			(effects
-				(font
-					(size 1.27 1.27)
-				)
+			(at 80.01 35.5599 90)
+			(effects
+				(font
+					(size 1.27 1.27)
+				)
+				(justify left)
 			)
 		)
 		(property "Value" "TLP175A"
-			(at 105.41 39.37 0)
-			(effects
-				(font
-					(size 1.27 1.27)
-				)
+			(at 80.01 38.0999 90)
+			(effects
+				(font
+					(size 1.27 1.27)
+				)
+				(justify left)
 			)
 		)
 		(property "Footprint" "Package_SO:MFSOP6-4_4.4x3.6mm_P1.27mm"
-			(at 105.41 53.34 0)
+			(at 67.31 36.83 0)
 			(effects
 				(font
@@
 		)
 		(property "Datasheet" "https://toshiba.semicon-storage.com/info/docget.jsp?did=13665&prodName=TLP175A"
-			(at 105.41 45.72 0)
+			(at 74.93 36.83 0)
 			(effects
 				(font
@@
 		)
 		(property "Description" "MOSFET Photorelay 1-Form-A, Voff 60V, Ion 100mA, SOP6"
-			(at 105.41 45.72 0)
-			(effects
-				(font
+			(at 74.93 36.83 0)
+			(effects
+				(font
