File: 2024/l2/l2.kicad_sch (KiCad schematic)
At the start: 20 parts, among them J1 Conn_01x04, J2 Conn_01x02, J3 Conn_01x04, U5 DEV-15583

Commit message: 5/9 final
fixed the problem with motor driver schematics
Connections:
- no-connect marks 16 -> 31
Changed lines of the file:
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@@
 	(paper "A4")
+	(no_connect
+		(at 203.2 87.63)
+	)
 	(no_connect
 		(at 222.25 139.7)
@@
 	)
 	(no_connect
+		(at 238.76 52.07)
+	)
+	(no_connect
+		(at 238.76 49.53)
+	)
+	(no_connect
+		(at 238.76 67.31)
+	)
+	(no_connect
+		(at 238.76 46.99)
+	)
+	(no_connect
+		(at 238.76 82.55)
+	)
+	(no_connect
 		(at 153.67 139.7)
 	)
@@
 	)
 	(no_connect
+		(at 238.76 69.85)
+	)
+	(no_connect
+		(at 238.76 85.09)
+	)
+	(no_connect
+		(at 238.76 59.69)
+	)
+	(no_connect
+		(at 238.76 57.15)
+	)
+	(no_connect
 		(at 153.67 132.08)
 	)
 	(no_connect
 		(at 153.67 114.3)
+	)
+	(no_connect
+		(at 238.76 62.23)
+	)
+	(no_connect
+		(at 203.2 82.55)
+	)
+	(no_connect
+		(at 238.76 64.77)
 	)
 	(no_connect
@@
 		(at 176.53 123.19)
 	)
+	(no_connect
+		(at 203.2 85.09)
+	)
+	(no_connect
+		(at 238.76 54.61)
+	)
 	(wire

Commit message: final 0.9
Connections:
- net INA_1: now also U5.9; no longer U5.2
- net INA_2: now also U5.17; no longer U5.5
- net INA_3: now also U5.15; no longer U5.10
- net INA_4: now also U5.10; no longer U5.13
- net INB_1: now also U5.5; no longer U5.3
- net INB_2: now also U5.19; no longer U5.6
- net INB_3: now also U5.13; no longer U5.11
- net INB_4: now also U5.12; no longer U5.14
- net PWM_1: now also U5.6; no longer U5.4
- net PWM_2: now also U5.18; no longer U5.9
- net PWM_3: now also U5.14; no longer U5.12
- net PWM_4: now also U5.11; no longer U5.15
- net RXL1: now also U5.21; no longer U5.0
- net RXL3: now also U5.0; no longer U5.7
- net TXL1: now also U5.20; no longer U5.1
- net TXL3: now also U5.1; no longer U5.8
- no-connect marks 31 -> 26
