File: 2024/l2/l2.kicad_pcb (KiCad board)
At the start: 2 copper layers, 175 x 169.4 mm, 38 parts, among them J1 Conn_01x04, J2 Conn_01x02, J3 Conn_01x04, J4 Conn_01x02, J5 Conn_01x02, J6 Conn_01x02, J7 Conn_01x02, Q1 IRF540N, Q2 IRF540N, Q3 IRF540N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

Commit message: v1.090
Parts:
- U1, U2, U3, U4: footprint Package_SO:ST_MultiPowerSO-30 -> Board:VNH5019A-E_SO-30
- moved U2 8.76 mm to (84.6, 70.3), turned to -132 degrees
- moved Q2 8.70 mm to (95.5, 60.2), turned to 138 degrees
- moved J5 3.14 mm to (98.5, 73.1)
- moved C2 1.87 mm to (91.6, 47.4), turned to 138 degrees
Routing:
- net /Motor Driver/MD: track 377.3 -> 224.3 mm
- net +12V: track 336.4 -> 220.8 mm
- net INB_1: track 136.1 -> 167.9 mm
- net INA_1: track 116.9 -> 146.0 mm
- net INA_2: track 114.0 -> 142.9 mm
- net PWM_1: track 130.9 -> 159.8 mm
- net PWM_2: track 119.4 -> 146.4 mm
- net INB_2: track 123.0 -> 147.2 mm
- net INB_4: track 27.8 -> 22.5 mm
- net PWM_4: track 29.8 -> 28.3 mm
- net /Motor Driver/CP1: track 12.6 -> 13.8 mm
- net GND: vias 0 -> 249
- added copper zone on B.Cu, net Net-(J4-Pin_1)
- added copper zone on B.Cu, net Net-(J4-Pin_2)
- added copper zone on B.Cu, net Net-(J5-Pin_1)
- added copper zone on B.Cu, net Net-(J5-Pin_2)
- added copper zone on B.Cu, net Net-(J6-Pin_1)
- added copper zone on B.Cu, net Net-(J6-Pin_2)
- added copper zone on B.Cu, net Net-(J7-Pin_1)
- added copper zone on B.Cu, net Net-(J7-Pin_2)
- added copper zone on B.Cu, net Net-(Q1-D)
- added copper zone on B.Cu, net Net-(Q2-D)
- added copper zone on B.Cu, net Net-(Q3-D)
- added copper zone on B.Cu, net Net-(Q4-D)
