File: 2024/l2/l2MotorDriver.kicad_sch (KiCad schematic)
At the start: 18 parts, among them J4 Conn_01x02, J5 Conn_01x02, J6 Conn_01x02, J7 Conn_01x02, Q1 IRF540N, Q2 IRF540N, Q3 IRF540N, Q4 IRF540N, SW1 SW_SPDT, U1 VNH5019A-E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

Commit message: v1.090
Parts:
- U1, U2, U3, U4: footprint Package_SO:ST_MultiPowerSO-30 -> Board:VNH5019A-E_SO-30
Changed lines of the file:
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@@
 			)
 		)
-		(property "Footprint" "Package_SO:ST_MultiPowerSO-30"
+		(property "Footprint" "Board:VNH5019A-E_SO-30"
 			(at 214.63 78.74 0)
 			(effects
@@
 			)
 		)
-		(property "Footprint" "Package_SO:ST_MultiPowerSO-30"
+		(property "Footprint" "Board:VNH5019A-E_SO-30"
 			(at 114.3 142.24 0)
 			(effects
@@
 			)
 		)
-		(property "Footprint" "Package_SO:ST_MultiPowerSO-30"
+		(property "Footprint" "Board:VNH5019A-E_SO-30"
 			(at 219.71 139.7 0)
 			(effects
@@
 			)
 		)
-		(property "Footprint" "Package_SO:ST_MultiPowerSO-30"
+		(property "Footprint" "Board:VNH5019A-E_SO-30"
 			(at 110.49 77.47 0)
 			(effects
