File: l2/l2.kicad_pcb (KiCad board)
At the start: 2 copper layers, 175 x 169.4 mm, 38 parts, among them J1 Conn_01x04, J2 Conn_01x02, J3 Conn_01x04, J4 Conn_01x02, J5 Conn_01x02, J6 Conn_01x02, J7 Conn_01x02, Q1 IRF540N, Q2 IRF540N, Q3 IRF540N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

Commit message: v2.0
l2 l3 done for print
Parts:
- SW1: footprint Button_Switch_THT:SS12D00G3-2.5mm -> Connector_JST:JST_XH_B3B-XH-AM_1x03_P2.50mm_Vertical
- moved R1 105.1 mm to (190.0, 97.3), turned to -90 degrees
- moved SW1 103.1 mm to (184.5, 95.9), turned to 90 degrees
Routing:
- net +5V: track 69.3 -> 165.3 mm, vias 0 -> 1
- net /Motor Driver/MD: track 225.2 -> 265.2 mm
- net Net-(SW1-A): track 2.63 -> 5.68 mm
- net GND: vias 205 -> 124
Other:
- outline, holes or cut-outs redrawn

Commit message: v2.1
fixed some stuff
Routing:
- net /Motor Driver/MD: track 265.2 -> 257.1 mm
- net +12V: track 220.8 -> 217.2 mm
- net GND: vias 124 -> 121
