File: l2/l2.kicad_sch (KiCad schematic)
At the start: 20 parts, among them J1 Conn_01x04, J2 Conn_01x02, J3 Conn_01x04, U5 DEV-15583

Commit message: v2.1
fixed some stuff
Connections:
- no-connect marks 26 -> 29
Changed lines of the file:
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@@
+	)
+	(no_connect
+		(at 203.2 57.15)
 	)
 	(no_connect
 		(at 238.76 46.99)
+	)
+	(no_connect
+		(at 203.2 52.07)
 	)
 	(no_connect
@@
 	)
 	(no_connect
+		(at 203.2 54.61)
+	)
+	(no_connect
