File: l2/l2MotorDriver.kicad_sch (KiCad schematic)
At the start: 18 parts, among them J4 Conn_01x02, J5 Conn_01x02, J6 Conn_01x02, J7 Conn_01x02, Q1 IRF540N, Q2 IRF540N, Q3 IRF540N, Q4 IRF540N, SW1 SW_SPDT, U1 VNH5019A-E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

Commit message: v2.0
l2 l3 done for print
Parts:
- SW1: footprint Button_Switch_THT:SS12D00G3-2.5mm -> Connector_JST:JST_XH_B3B-XH-AM_1x03_P2.50mm_Vertical
Changed lines of the file:
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@@
 					(size 1.27 1.27)
 				)
+				(hide yes)
 			)
 		)
-		(property "Footprint" "Button_Switch_THT:SS12D00G3-2.5mm"
+		(property "Footprint" "Connector_JST:JST_XH_B3B-XH-AM_1x03_P2.50mm_Vertical"
 			(at 82.55 175.26 0)
 			(effects
